File: ecad/UPS/UPSOutput.kicad_sch (KiCad schematic)
At the start: 18 parts, among them U2 MPQ5031GRE-0001-AEC1-P

Commit message: Made Buck Convertor Schematic
Parts:
- U2: footprint QFN-20_MPQ5031_MNP -> UPS:QFN-20_MPQ5031_MNP
Changed lines of the file:
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@@
 			)
 		)
-		(property "Footprint" "QFN-20_MPQ5031_MNP"
+		(property "Footprint" "UPS:QFN-20_MPQ5031_MNP"
 			(at 67.31 64.77 0)
 			(effects
