File: ecad/UPS/UPSOutput.kicad_sch (KiCad schematic)
At the start: 21 parts, among them Q6 IRLR7843TRPBF, U2 MPQ5031GRE-0001-AEC1-P, U3 L78L05_SOT89

Commit message: Add footprints for USB receptacle
Parts:
- J1: renamed from USB_Output1; footprint (none) -> Connector_USB:USB_C_Receptacle_GCT_USB4110
- renumbered C7 to C?, C9 to C?, C6 to C?, C10 to C?, C11 to C?, C5 to C?, C8 to C?, C12 to C?, D4 to D?, D3 to D?, D5 to D?, D1 to D?, D2 to D?, Q6 to Q?, R7 to R?, R6 to R?, R8 to R?, TH1 to TH?, U2 to U1, U3 to U?
Connections:
- net GND: now also J1.S1 (SHIELD)
Changed lines of the file:
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@@
 	(wire
 		(pts
+			(xy 251.46 31.75) (xy 251.46 27.94)
+		)
+		(stroke
+			(width 0)
+			(type default)
+		)
+	)
+	(wire
+		(pts
 			(xy 162.56 62.23) (xy 162.56 71.12)
 		)
@@
 		(on_board yes)
 		(dnp no)
-		(property "Reference" "C7"
+		(property "Reference" "C?"
 			(at 207.01 73.6599 0)
 			(effects
@@
 		(dnp no)
 		(fields_autoplaced yes)
-		(property "Reference" "#PWR0102"
+		(property "Reference" "#PWR03"
 			(at 66.04 33.02 0)
 			(effects
@@
 		(dnp no)
 		(fields_autoplaced yes)
-		(property "Reference" "U3"
+		(property "Reference" "U?"
 			(at 43.18 114.2999 90)
 			(effects
@@
 		)
 		(instances
+			(project "UPSOutput"
+				(path "/917f3576-2b89-40c4-9175-933056884ccc"
+					(reference "U?")
+					(unit 1)
+				)
+			)
 			(project "UPS"
 				(path "/9d92b60a-4a6b-449c-b462-cab19e69d38c/c2035c51-7de6-43a1-947f-d073f8318def"
@@
 		(on_board yes)
 		(dnp no)
-		(property "Reference" "R7"
+		(property "Reference" "R?"
 			(at 142.24 50.292 90)
 			(effects
@@
 		(on_board yes)
 		(dnp no)
-		(property "Reference" "D4"
+		(property "Reference" "D?"
 			(at 195.58 76.2001 90)
 			(effects
@@
 		(dnp no)
 		(fields_autoplaced yes)
-		(property "Reference" "#PWR09"
+		(property "Reference" "#PWR?"
 			(at 182.88 91.44 0)
 			(effects
@@
 		(on_board yes)
 		(dnp no)
-		(property "Reference" "D3"
+		(property "Reference" "D?"
 			(at 185.42 76.2001 90)
 			(effects
@@
 		(on_board yes)
 		(dnp no)
-		(property "Reference" "R6"
+		(property "Reference" "R?"
 			(at 142.24 43.688 90)
 			(effects
@@
 		(dnp no)
 		(fields_autoplaced yes)
-		(property "Reference" "C9"
+		(property "Reference" "C?"
 			(at 68.58 73.6599 0)
 			(effects
@@
 		(on_board yes)
 		(dnp no)
-		(property "Reference" "U2"
+		(property "Reference" "U1"
 			(at 92.71 74.93 0)
 			(effects
@@
 		(dnp no)
 		(fields_autoplaced yes)
-		(property "Reference" "#PWR010"
+		(property "Reference" "#PWR?"
 			(at 198.12 91.44 0)
 			(effects
@@
 		(on_board yes)
 		(dnp no)
-		(property "Reference" "C6"
+		(property "Reference" "C?"
 			(at 123.19 68.834 0)
 			(effects
@@
 		(dnp no)
 		(fields_autoplaced yes)
-		(property "Reference" "#PWR0104"
+		(property "Reference" "#PWR01"
 			(at 243.84 21.59 0)
 			(effects
@@
 		(dnp no)
 		(fields_autoplaced yes)
-		(property "Reference" "#PWR0108"
+		(property "Reference" "#PWR?"
 			(at 39.37 124.46 0)
 			(effects
@@
 		)
 		(instances
+			(project "UPSOutput"
+				(path "/917f3576-2b89-40c4-9175-933056884ccc"
+					(reference "#PWR?")
+					(unit 1)
+				)
+			)
 			(project "UPS"
 				(path "/9d92b60a-4a6b-449c-b462-cab19e69d38c/c2035c51-7de6-43a1-947f-d073f8318def"
@@
 		(dnp no)
 		(fields_autoplaced yes)
-		(property "Reference" "#PWR011"
+		(property "Reference" "#PWR?"
 			(at 113.03 25.4 0)
 			(effects
@@
 		(on_board yes)
 		(dnp no)
-		(property "Reference" "C10"
+		(property "Reference" "C?"
 			(at 53.34 73.6599 0)
 			(effects
@@
 		(dnp no)
 		(fields_autoplaced yes)
-		(property "Reference" "#PWR08"
+		(property "Reference" "#PWR?"
 			(at 158.75 91.44 0)
 			(effects
@@
 	)
 	(symbol
+		(lib_id "power:GND")
+		(at 251.46 27.94 180)
+		(unit 1)
+		(exclude_from_sim no)
+		(in_bom yes)
+		(on_board yes)
+		(dnp no)
+		(fields_autoplaced yes)
+		(property "Reference" "#PWR05"
+			(at 251.46 21.59 0)
+			(effects
+				(font
+					(size 1.27 1.27)
+				)
+				(hide yes)
+			)
+		)
+		(property "Value" "GND"
+			(at 251.46 22.86 0)
+			(effects
+				(font
+					(size 1.27 1.27)
+				)
+			)
+		)
+		(property "Footprint" ""
+			(at 251.46 27.94 0)
+			(effects
+				(font
+					(size 1.27 1.27)
+				)
+				(hide yes)
+			)
+		)
+		(property "Datasheet" ""
+			(at 251.46 27.94 0)
+			(effects
+				(font
+					(size 1.27 1.27)
+				)
+				(hide yes)
+			)
+		)
+		(property "Description" "Power symbol creates a global label with name \"GND\" , ground"
+			(at 251.46 27.94 0)
+			(effects
+				(font
+					(size 1.27 1.27)
+				)
+				(hide yes)
+			)
+		)
+		(pin "1"
+		)
+		(instances
+			(project "UPSOutput"
+				(path "/917f3576-2b89-40c4-9175-933056884ccc"
+					(reference "#PWR05")
+					(unit 1)
+				)
+			)
+		)
+	)
+	(symbol
 		(lib_id "Device:C")
 		(at 139.7 82.55 90)
@@
 		(dnp no)
 		(fields_autoplaced yes)
-		(property "Reference" "C11"
+		(property "Reference" "C?"
 			(at 139.7 74.93 90)
 			(effects
@@
 		(dnp no)
 		(fields_autoplaced yes)
-		(property "Reference" "#PWR013"
+		(property "Reference" "#PWR?"
 			(at 245.11 85.09 0)
 			(effects
@@
 		(dnp no)
 		(fields_autoplaced yes)
-		(property "Reference" "Q6"
+		(property "Reference" "Q?"
 			(at 113.03 106.68 90)
 			(effects
@@
 		)
 		(instances
+			(project "UPSOutput"
+				(path "/917f3576-2b89-40c4-9175-933056884ccc"
+					(reference "Q?")
+					(unit 1)
+				)
+			)
 			(project ""
 				(path "/9d92b60a-4a6b-449c-b462-cab19e69d38c/c2035c51-7de6-43a1-947f-d073f8318def"
@@
 		(dnp no)
 		(fields_autoplaced yes)
-		(property "Reference" "#PWR0106"
+		(property "Reference" "#PWR?"
 			(at 20.32 115.57 0)
 			(effects
@@
 		)
 		(instances
+			(project "UPSOutput"
+				(path "/917f3576-2b89-40c4-9175-933056884ccc"
+					(reference "#PWR?")
+					(unit 1)
+				)
+			)
 			(project "UPS"
 				(path "/9d92b60a-4a6b-449c-b462-cab19e69d38c/c2035c51-7de6-43a1-947f-d073f8318def"
@@
 		(on_board yes)
 		(dnp no)
-		(property "Reference" "D5"
+		(property "Reference" "D?"
 			(at 232.4101 92.71 90)
 			(effects
@@
 		)
 		(instances
+			(project "UPSOutput"
+				(path "/917f3576-2b89-40c4-9175-933056884ccc"
+					(reference "D?")
+					(unit 1)
+				)
+			)
 			(project "UPS"
 				(path "/9d92b60a-4a6b-449c-b462-cab19e69d38c/c2035c51-7de6-43a1-947f-d073f8318def"
@@
 		(dnp no)
 		(fields_autoplaced yes)
-		(property "Reference" "#PWR012"
+		(property "Reference" "#PWR?"
 			(at 149.86 25.4 0)
 			(effects
@@
 		(dnp no)
 		(fields_autoplaced yes)
-		(property "Reference" "#PWR0101"
+		(property "Reference" "#PWR02"
 			(at 118.11 82.55 0)
 			(effects
@@
 		(dnp no)
 		(fields_autoplaced yes)
-		(property "Reference" "D1"
+		(property "Reference" "D?"
 			(at 156.21 73.6599 90)
 			(effects
@@
 		(on_board yes)
 		(dnp no)
-		(property "Reference" "D2"
+		(property "Reference" "D?"
 			(at 165.1 73.6599 90)
 			(effects
@@
 		(dnp no)
 		(fields_autoplaced yes)
-		(property "Reference" "C5"
+		(property "Reference" "C?"
 			(at 138.43 68.5799 0)
 			(effects
@@
 		(dnp no)
 		(fields_autoplaced yes)
-		(property "Reference" "#PWR0103"
+		(property "Reference" "#PWR04"
 			(at 60.96 90.17 0)
 			(effects
@@
 		(dnp no)
 		(fields_autoplaced yes)
-		(property "Reference" "R8"
+		(property "Reference" "R?"
 			(at 118.11 19.05 90)
 			(effects
@@
 		(dnp no)
 		(fields_autoplaced yes)
-		(property "Reference" "C8"
+		(property "Reference" "C?"
 			(at 173.99 73.6599 0)
 			(effects
@@
 		(dnp no)
 		(fields_autoplaced yes)
-		(property "Reference" "#PWR0107"
+		(property "Reference" "#PWR?"
 			(at 48.26 41.91 0)
 			(effects
@@
 		)
 		(instances
+			(project "UPSOutput"
+				(path "/917f3576-2b89-40c4-9175-933056884ccc"
+					(reference "#PWR?")
+					(unit 1)
+				)
+			)
 			(project "UPS"
 				(path "/9d92b60a-4a6b-449c-b462-cab19e69d38c/c2035c51-7de6-43a1-947f-d073f8318def"
@@
 		(dnp no)
 		(fields_autoplaced yes)
-		(property "Reference" "USB_Output1"
+		(property "Reference" "J1"
 			(at 255.27 53.3399 0)
 			(effects
@@
 			)
 		)
-		(property "Footprint" ""
+		(property "Footprint" "Connector_USB:USB_C_Receptacle_GCT_USB4110"
 			(at 240.03 54.61 0)
 			(effects
@@
 		(on_board yes)
 		(dnp no)
-		(property "Reference" "TH1"
+		(property "Reference" "TH?"
 			(at 133.6675 19.05 90)
 			(effects
@@
 		(dnp no)
 		(fields_autoplaced yes)
-		(property "Reference" "C12"
+		(property "Reference" "C?"
 			(at 231.14 77.47 90)
 			(effects

Commit message: Fix duplicate component names.
Parts:
- removed Q?: IRLR7843TRPBF, Package_TO_SOT_SMD:TO-252-2, symbol Transistor_FET:Q_NMOS_GDS
- added Q3: IRLR7843TRPBF, Package_TO_SOT_SMD:TO-252-2, symbol Transistor_FET:Q_NMOS_GDS
- gave numbers to parts that had none: 18
- renumbered J1 to J3, U1 to U2
Connections:
- net vbus: now also Q3.3 (S)
- net at U2.19 (VDRV): now also Q3.1 (G)
- net at C11.2, C12.1, D5.1 (K)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: now also Q3.2 (D)
Changed lines of the file:
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@@
 		(on_board yes)
 		(dnp no)
-		(property "Reference" "C?"
+		(property "Reference" "C7"
 			(at 207.01 73.6599 0)
 			(effects
@@
 		(dnp no)
 		(fields_autoplaced yes)
-		(property "Reference" "#PWR03"
+		(property "Reference" "#PWR0102"
 			(at 66.04 33.02 0)
 			(effects
@@
 		(dnp no)
 		(fields_autoplaced yes)
-		(property "Reference" "U?"
+		(property "Reference" "U3"
 			(at 43.18 114.2999 90)
 			(effects
@@
 		(on_board yes)
 		(dnp no)
-		(property "Reference" "R?"
+		(property "Reference" "R7"
 			(at 142.24 50.292 90)
 			(effects
@@
 		(on_board yes)
 		(dnp no)
-		(property "Reference" "D?"
+		(property "Reference" "D4"
 			(at 195.58 76.2001 90)
 			(effects
@@
 		(dnp no)
 		(fields_autoplaced yes)
-		(property "Reference" "#PWR?"
+		(property "Reference" "#PWR09"
 			(at 182.88 91.44 0)
 			(effects
@@
 		(on_board yes)
 		(dnp no)
-		(property "Reference" "D?"
+		(property "Reference" "D3"
 			(at 185.42 76.2001 90)
 			(effects
@@
 		(on_board yes)
 		(dnp no)
-		(property "Reference" "R?"
+		(property "Reference" "R6"
 			(at 142.24 43.688 90)
 			(effects
@@
 		(dnp no)
 		(fields_autoplaced yes)
-		(property "Reference" "C?"
+		(property "Reference" "C9"
 			(at 68.58 73.6599 0)
 			(effects
@@
 		(on_board yes)
 		(dnp no)
-		(property "Reference" "U1"
+		(property "Reference" "U2"
 			(at 92.71 74.93 0)
 			(effects
@@
 		(dnp no)
 		(fields_autoplaced yes)
-		(property "Reference" "#PWR?"
+		(property "Reference" "#PWR010"
 			(at 198.12 91.44 0)
 			(effects
@@
 		(on_board yes)
 		(dnp no)
-		(property "Reference" "C?"
+		(property "Reference" "C6"
 			(at 123.19 68.834 0)
 			(effects
@@
 		(dnp no)
 		(fields_autoplaced yes)
-		(property "Reference" "#PWR01"
+		(property "Reference" "#PWR0104"
 			(at 243.84 21.59 0)
 			(effects
@@
 		(dnp no)
 		(fields_autoplaced yes)
-		(property "Reference" "#PWR?"
+		(property "Reference" "#PWR0108"
 			(at 39.37 124.46 0)
 			(effects
@@
 		(dnp no)
 		(fields_autoplaced yes)
-		(property "Reference" "#PWR?"
+		(property "Reference" "#PWR011"
 			(at 113.03 25.4 0)
 			(effects
@@
 				(path "/9d92b60a-4a6b-449c-b462-cab19e69d38c/c2035c51-7de6-43a1-947f-d073f8318def"
 					(reference "#PWR011")
+					(unit 1)
+				)
+			)
+		)
+	)
+	(symbol
+		(lib_id "Transistor_FET:Q_NMOS_GDS")
+		(at 113.03 100.33 270)
+		(unit 1)
+		(exclude_from_sim no)
+		(in_bom yes)
+		(on_board yes)
+		(dnp no)
+		(fields_autoplaced yes)
+		(property "Reference" "Q3"
+			(at 113.03 106.68 90)
+			(effects
+				(font
+					(size 1.27 1.27)
+				)
+			)
+		)
+		(property "Value" "IRLR7843TRPBF"
+			(at 113.03 109.22 90)
+			(effects
+				(font
+					(size 1.27 1.27)
+				)
+			)
+		)
+		(property "Footprint" "Package_TO_SOT_SMD:TO-252-2"
+			(at 115.57 105.41 0)
+			(effects
+				(font
+					(size 1.27 1.27)
+				)
+				(hide yes)
+			)
+		)
+		(property "Datasheet" "~"
+			(at 113.03 100.33 0)
+			(effects
+				(font
+					(size 1.27 1.27)
+				)
+				(hide yes)
+			)
+		)
+		(property "Description" "N-MOSFET transistor, gate/drain/source"
+			(at 113.03 100.33 0)
+			(effects
+				(font
+					(size 1.27 1.27)
+				)
+				(hide yes)
+			)
+		)
+		(pin "1"
+		)
+		(pin "3"
+		)
+		(pin "2"
+		)
+		(instances
+			(project "UPS"
+				(path "/9d92b60a-4a6b-449c-b462-cab19e69d38c/c2035c51-7de6-43a1-947f-d073f8318def"
+					(reference "Q3")
 					(unit 1)
 				)
@@
 		(on_board yes)
 		(dnp no)
-		(property "Reference" "C?"
+		(property "Reference" "C10"
 			(at 53.34 73.6599 0)
 			(effects
@@
 		(dnp no)
 		(fields_autoplaced yes)
-		(property "Reference" "#PWR?"
+		(property "Reference" "#PWR08"
 			(at 158.75 91.44 0)
 			(effects
@@
 		(dnp no)
 		(fields_autoplaced yes)
-		(property "Reference" "#PWR05"
+		(property "Reference" "#PWR0117"
 			(at 251.46 21.59 0)
 			(effects
@@
 				)
 			)
+			(project "UPS"
+				(path "/9d92b60a-4a6b-449c-b462-cab19e69d38c/c2035c51-7de6-43a1-947f-d073f8318def"
+					(reference "#PWR0117")
+					(unit 1)
+				)
+			)
 		)
 	)
@@
 		(dnp no)
 		(fields_autoplaced yes)
-		(property "Reference" "C?"
+		(property "Reference" "C11"
 			(at 139.7 74.93 90)
 			(effects
@@
 		(dnp no)
 		(fields_autoplaced yes)
-		(property "Reference" "#PWR?"
+		(property "Reference" "#PWR013"
 			(at 245.11 85.09 0)
 			(effects
@@
 	)
 	(symbol
-		(lib_id "Transistor_FET:Q_NMOS_GDS")
-		(at 113.03 100.33 270)
-		(unit 1)
-		(exclude_from_sim no)
-		(in_bom yes)
-		(on_board yes)
-		(dnp no)
-		(fields_autoplaced yes)
-		(property "Reference" "Q?"
-			(at 113.03 106.68 90)
-			(effects
-				(font
-					(size 1.27 1.27)
-				)
-			)
-		)
-		(property "Value" "IRLR7843TRPBF"
-			(at 113.03 109.22 90)
-			(effects
-				(font
-					(size 1.27 1.27)
-				)
-			)
-		)
-		(property "Footprint" "Package_TO_SOT_SMD:TO-252-2"
-			(at 115.57 105.41 0)
-			(effects
-				(font
-					(size 1.27 1.27)
-				)
-				(hide yes)
-			)
-		)
-		(property "Datasheet" "~"
-			(at 113.03 100.33 0)
-			(effects
-				(font
-					(size 1.27 1.27)
-				)
-				(hide yes)
-			)
-		)
-		(property "Description" "N-MOSFET transistor, gate/drain/source"
-			(at 113.03 100.33 0)
-			(effects
-				(font
-					(size 1.27 1.27)
-				)
-				(hide yes)
-			)
-		)
-		(pin "1"
-		)
-		(pin "3"
-		)
-		(pin "2"
-		)
-		(instances
-			(project "UPSOutput"
-				(path "/917f3576-2b89-40c4-9175-933056884ccc"
-					(reference "Q?")
-					(unit 1)
-				)
-			)
-			(project ""
-				(path "/9d92b60a-4a6b-449c-b462-cab19e69d38c/c2035c51-7de6-43a1-947f-d073f8318def"
-					(reference "Q6")
-					(unit 1)
-				)
-			)
-		)
-	)
-	(symbol
 		(lib_id "power:GND")
 		(at 26.67 115.57 270)
@@
 		(dnp no)
 		(fields_autoplaced yes)
-		(property "Reference" "#PWR?"
+		(property "Reference" "#PWR0106"
 			(at 20.32 115.57 0)
 			(effects
@@
 		(on_board yes)
 		(dnp no)
-		(property "Reference" "D?"
+		(property "Reference" "D5"
 			(at 232.4101 92.71 90)
 			(effects
@@
 		(dnp no)
 		(fields_autoplaced yes)
-		(property "Reference" "#PWR?"
+		(property "Reference" "#PWR012"
 			(at 149.86 25.4 0)
 			(effects
@@
 		(dnp no)
 		(fields_autoplaced yes)
-		(property "Reference" "#PWR02"
+		(property "Reference" "#PWR0101"
 			(at 118.11 82.55 0)
 			(effects
@@
 		(dnp no)
 		(fields_autoplaced yes)
-		(property "Reference" "D?"
+		(property "Reference" "D1"
 			(at 156.21 73.6599 90)
 			(effects
@@
 		(on_board yes)
 		(dnp no)
-		(property "Reference" "D?"
+		(property "Reference" "D2"
 			(at 165.1 73.6599 90)
 			(effects
@@
 		(dnp no)
 		(fields_autoplaced yes)
-		(property "Reference" "C?"
+		(property "Reference" "C5"
 			(at 138.43 68.5799 0)
 			(effects
@@
 		(dnp no)
 		(fields_autoplaced yes)
-		(property "Reference" "#PWR04"
+		(property "Reference" "#PWR0103"
 			(at 60.96 90.17 0)
 			(effects
@@
 		(dnp no)
 		(fields_autoplaced yes)
-		(property "Reference" "R?"
+		(property "Reference" "R8"
 			(at 118.11 19.05 90)
 			(effects
@@
 		(dnp no)
 		(fields_autoplaced yes)
-		(property "Reference" "C?"
+		(property "Reference" "C8"
 			(at 173.99 73.6599 0)
 			(effects
@@
 		(dnp no)
 		(fields_autoplaced yes)
-		(property "Reference" "#PWR?"
+		(property "Reference" "#PWR0107"
 			(at 48.26 41.91 0)
 			(effects
@@
 		(dnp no)
 		(fields_autoplaced yes)
-		(property "Reference" "J1"
+		(property "Reference" "J3"
 			(at 255.27 53.3399 0)
 			(effects
@@
 			(project "UPS"
 				(path "/9d92b60a-4a6b-449c-b462-cab19e69d38c/c2035c51-7de6-43a1-947f-d073f8318def"
-					(reference "USB_Output1")
+					(reference "J3")
 					(unit 1)
 				)
@@
 		(on_board yes)
 		(dnp no)
-		(property "Reference" "TH?"
+		(property "Reference" "TH1"
 			(at 133.6675 19.05 90)
 			(effects
@@
 		(dnp no)
 		(fields_autoplaced yes)
-		(property "Reference" "C?"
+		(property "Reference" "C12"
 			(at 231.14 77.47 90)
 			(effects

Commit message: Add caps to regulator
Parts:
- added C59: 330nF, symbol Device:C
- added C60: 100nF, symbol Device:C
- added TP6: VBus, TestPoint:TestPoint_Pad_D1.5mm, symbol Connector:TestPoint
- added TP7: NTC1, TestPoint:TestPoint_Pad_D1.5mm, symbol Connector:TestPoint
- added TP8: 5V_REG, TestPoint:TestPoint_Pad_D1.5mm, symbol Connector:TestPoint
Connections:
- net +5V: now also C60.2, TP8.1
- net GND: now also C59.2, C60.1
- net vbus: now also C59.1
- net at R8.2, TH1.1, U2.13 (NTC): now also TP7.1
- net at C11.2, C12.1, D5.1 (K)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: now also TP6.1

Commit message: added components to bom
Parts:
- C10, C11, C12, C60: footprint (none) -> Capacitor_SMD:C_0805_2012Metric_Pad1.18x1.45mm_HandSolder
- C5, C59, C6, C7, C8, C9: footprint (none) -> Capacitor_SMD:C_0603_1608Metric_Pad1.08x0.95mm_HandSolder
Changed lines of the file:
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@@
 			)
 		)
-		(property "Footprint" ""
+		(property "Footprint" "Capacitor_SMD:C_0603_1608Metric_Pad1.08x0.95mm_HandSolder"
 			(at 204.1652 78.74 0)
 			(effects
@@
 			)
 		)
-		(property "Footprint" ""
+		(property "Footprint" "Capacitor_SMD:C_0603_1608Metric_Pad1.08x0.95mm_HandSolder"
 			(at 30.1752 115.57 0)
 			(effects
@@
 			)
 		)
-		(property "Footprint" ""
+		(property "Footprint" "Capacitor_SMD:C_0603_1608Metric_Pad1.08x0.95mm_HandSolder"
 			(at 65.7352 78.74 0)
 			(effects
@@
 			)
 		)
-		(property "Footprint" ""
+		(property "Footprint" "Capacitor_SMD:C_0603_1608Metric_Pad1.08x0.95mm_HandSolder"
 			(at 130.5052 73.66 0)
 			(effects
@@
 			)
 		)
-		(property "Footprint" ""
+		(property "Footprint" "Capacitor_SMD:C_0805_2012Metric_Pad1.18x1.45mm_HandSolder"
 			(at 56.1848 78.74 0)
 			(effects
@@
 			)
 		)
-		(property "Footprint" ""
+		(property "Footprint" "Capacitor_SMD:C_0805_2012Metric_Pad1.18x1.45mm_HandSolder"
 			(at 143.51 81.5848 0)
 			(effects
@@
 			)
 		)
-		(property "Footprint" ""
+		(property "Footprint" "Capacitor_SMD:C_0603_1608Metric_Pad1.08x0.95mm_HandSolder"
 			(at 135.5852 73.66 0)
 			(effects
@@
 			)
 		)
-		(property "Footprint" ""
+		(property "Footprint" "Capacitor_SMD:C_0603_1608Metric_Pad1.08x0.95mm_HandSolder"
 			(at 176.8348 78.74 0)
 			(effects
@@
 			)
 		)
-		(property "Footprint" ""
+		(property "Footprint" "Capacitor_SMD:C_0805_2012Metric_Pad1.18x1.45mm_HandSolder"
 			(at 30.1752 128.27 0)
 			(effects
@@
 			)
 		)
-		(property "Footprint" ""
+		(property "Footprint" "Capacitor_SMD:C_0805_2012Metric_Pad1.18x1.45mm_HandSolder"
 			(at 234.95 84.1248 0)
 			(effects
